File: kancil-meter-vdo-73230-e.kicad_pcb (KiCad board)
At the start: 2 copper layers, 306 x 116 mm, 0 parts

Commit message: feat: Finish routing all traces
Signed-off-by: Andrew Yong <me@ndoo.sg>
Parts:
- added REF**: MountingHole_B8.5D_TopOnly, MountingHole:MountingHole_B8.5D_TopOnly, F.Cu at (313.0, 127.0)
- added REF**: MountingHole_B8.5D_TopOnly, MountingHole:MountingHole_B8.5D_TopOnly, F.Cu at (297.0, 156.0)
- added REF**: MountingHole_B8.5D_TopOnly, MountingHole:MountingHole_B8.5D_TopOnly, F.Cu at (183.0, 133.0)
- added REF**: MountingHole_B8.5D_TopOnly, MountingHole:MountingHole_B8.5D_TopOnly, F.Cu at (181.0, 104.0)
- added REF**: MountingHole_B8.5D_TopOnly, MountingHole:MountingHole_B8.5D_TopOnly, F.Cu at (87.0, 127.0)
- added REF**: MountingHole_B8.5D_TopOnly, MountingHole:MountingHole_B8.5D_TopOnly, F.Cu at (103.0, 156.0)
- added REF**: MountingHole_B8.5D_TopOnly, MountingHole:MountingHole_B8.5D_TopOnly, F.Cu at (220.0, 122.0)
- added REF**: MountingHole_B8.5D_TopOnly, MountingHole:MountingHole_B8.5D_TopOnly, F.Cu at (300.0, 120.0)
- added REF**: MountingHole_B8.5D_TopOnly, MountingHole:MountingHole_B8.5D_TopOnly, F.Cu at (219.0, 104.0)
- added REF**: MountingHole_B8.5D_TopOnly, MountingHole:MountingHole_B8.5D_TopOnly, F.Cu at (325.5, 136.0)
- added REF**: MountingHole_B8.5D_TopOnly, MountingHole:MountingHole_B8.5D_TopOnly, F.Cu at (100.0, 120.0)
- added REF**: MountingHole_B8.5D_TopOnly, MountingHole:MountingHole_B8.5D_TopOnly, F.Cu at (224.0, 182.0)
Other:
- board size 306 x 116 mm -> 305.8 x 116 mm

Commit message: feat: Silkscreen additions and cleanup
Signed-off-by: Andrew Yong <me@ndoo.sg>
Parts:
- added REF**: OSHW-Logo_7.5x8mm_SilkScreen, Symbol:OSHW-Logo_7.5x8mm_SilkScreen, F.Cu at (286.0, 186.5)
- added REF**: MountingHole_B8.5D_TopOnly, MountingHole:MountingHole_B8.5D_TopOnly, F.Cu at (200.0, 102.5)
Other:
- outline, holes or cut-outs redrawn
- board text added: "+"
- board text added: "A"
- board text added: "B"
- board text added: "CHECK ENGINE (EFI ONLY)"
- board text added: "FUEL SENDER"
- board text added: "GAUGE EARTH"
- board text added: "ILLUMINATION"
- board text added: "MADE ON EARTH BY HUMANS"
- board text added: "OIL PRESSURE"
- board text added: "OIL PRESSURE SW"
- board text added: "Perodua Kancil K2/K3 M/T Meter Flex © Andrew Yong, 2026"
- board text added: "TEMP SENDER"
- board text added: "TURN (LEFT)"
- board text added: "TURN (RIGHT)"
- board text removed: "221.2K"
- board text removed: "4"
- board text removed: "C.ENG"
- board text removed: "C1"
- board text removed: "C6"
- board text removed: "OIL"
- board text removed: "TURN-L"
- board text removed: "TURN-R"
